Commit message: pushing changes in src on 15/9/25

File: dojo/description/robot_core.xacro (robot description, xacro)
@@ -1,81 +1,94 @@
 <?xml version="1.0"?>
-<robot xmlns:xacro="http://www.ros.org/wiki/xacro">
+<robot xmlns:xacro="http://www.ros.org/wiki/xacro" >
     <xacro:include filename="inertial_macros.xacro"/>
-    <material name = "white">
-        <color rgba = "1 1 1 1"/>
+    <xacro:property name="chassis_length" value="0.250"/>
+    <xacro:property name="chassis_width" value="0.200"/>
+    <xacro:property name="chassis_height" value="0.072"/>
+    <xacro:property name="chassis_mass" value="1.0"/>
+    <xacro:property name="wheel_radius" value="0.0425"/>
+    <xacro:property name="wheel_thickness" value="0.038"/>
+    <xacro:property name="wheel_mass" value="0.05"/>
+    <xacro:property name="wheel_offset_x" value="0.216"/>
+    <xacro:property name="wheel_offset_y" value="0.123"/>
+    <xacro:property name="wheel_offset_z" value="0.01"/>
+    <xacro:property name="caster_wheel_radius" value="0.01"/>
+    <xacro:property name="caster_wheel_mass" value="0.01"/>
+    <xacro:property name="caster_wheel_offset_x" value="0.075"/>
+    <xacro:property name="caster_wheel_offset_z" value="${wheel_offset_z - wheel_radius + caster_wheel_radius}"/>
+    <material name="white">
+        <color rgba="1 1 1 1" />
     </material>
-    <material name = "orange">
-        <color rgba = "1 0.3 0.1 1"/>
+    <material name="orange">
+        <color rgba="1 0.3 0.1 1"/>
     </material>
-    <material name = "blue">
-        <color rgba = "0.3 0.3 1 1"/>
+    <material name="blue">
+        <color rgba="0.2 0.2 1 1"/>
     </material>
-    <material name = "black">
-        <color rgba = "0 0 0 1"/>
+    <material name="black">
+        <color rgba="0 0 0 1"/>
     </material>
-    <material name = "red">
-        <color rgba = "1 0 0 1"/>
+    <material name="red">
+        <color rgba="1 0 0 1"/>
     </material>
-    <!-- base link -->
-    <link name = "base_link">
+    <!-- BASE LINK -->
+    <link name="base_link">
     </link>
-    <!-- Base foot print -->
-     <joint name="base_footprint_joint" type="fixed">
+    <!-- BASE_FOOTPRINT LINK -->
+    <joint name="base_footprint_joint" type="fixed">
         <parent link="base_link"/>
-        <child link = "base_footprint"/>
-        <origin xyz = "0 0 0" rpy="0 0 0"/>
-     </joint>
-     <link name="base_footprint">
-     </link>
-    <!-- Chassis -->
-    <joint name = "chassis_joint" type="fixed">
+        <child link="base_footprint"/>
+        <origin xyz="0 0 0" rpy="0 0 0"/>
+    </joint>
+    <link name="base_footprint">
+    </link>
+    <!-- CHASSIS LINK -->
+    <joint name="chassis_joint" type="fixed">
         <parent link="base_link"/>
-        <child link = "chassis"/>
-        <origin xyz = "0 0 -0.07"/>
+        <child link="chassis"/>
+        <origin xyz="${-wheel_offset_x} 0 ${-wheel_offset_z}"/>
+         <!-- <origin xyz="${-wheel_offset_x} 0 ${-wheel_offset_z}" rpy="0 0 ${pi}"/> -->
     </joint>
     <link name="chassis">
         <visual>
-            <origin xyz = "0 0 0.035"/>
+            <origin xyz="${chassis_length/2} 0 ${chassis_height/2}"/>
             <geometry>
-                <cylinder radius = "0.125" length = "0.07"/>
+                <box size="${chassis_length} ${chassis_width} ${chassis_height}"/>
             </geometry>
-            <material name="white"/>
+            <material name="orange"/>
         </visual>
         <collision>
-            <origin xyz = "0 0 0.035"/>
+            <origin xyz="${chassis_length/2} 0 ${chassis_height/2}"/>
             <geometry>
-                <cylinder radius = "0.125" length = "0.07"/>
+                <box size="${chassis_length} ${chassis_width} ${chassis_height}"/>
             </geometry>
         </collision>
-        <xacro:inertial_cylinder mass= "0.5" radius="0.125" length="0.07">
-            <origin xyz="0.0 0.0 0.035" rpy="0.0 0.0 0.0"/>
-        </xacro:inertial_cylinder>
+        <xacro:inertial_box mass="0.5" x="${chassis_length}" y="${chassis_width}" z="${chassis_height}">
+            <origin xyz="${chassis_length/2} 0 ${chassis_height/2}" rpy="0 0 0"/>
+        </xacro:inertial_box>
     </link>
     <gazebo reference="chassis">
-        <material>Gazebo/White</material>
+        <material>Gazebo/Orange</material>
     </gazebo>
-    <!-- left wheel -->
-    <joint name = "left_wheel_joint" type="continuous">
+    <!-- LEFT WHEEL LINK -->
+    <joint name="left_wheel_joint" type="continuous">
         <parent link="base_link"/>
         <child link="left_wheel"/>
-        <origin xyz="0.0 0.14 -0.07" rpy="-${pi/2} 0.0 0.0"/>
-        <axis xyz="0.0 0.0 1"/>
+        <origin xyz="0 ${wheel_offset_y} 0" rpy="-${pi/2} 0 0" />
+        <axis xyz="0 0 1"/>
     </joint>
     <link name="left_wheel">
         <visual>
-            <origin xyz="0 0 0"/>
             <geometry>
-                <cylinder radius="0.0325" length="0.026"/>
+                <cylinder radius="${wheel_radius}" length="${wheel_thickness}"/>
             </geometry>
             <material name="blue"/>
         </visual>
         <collision>
-            <origin xyz="0 0 0"/>
             <geometry>
-                <sphere radius="0.0325"/>
+                <sphere radius="${wheel_radius}"/>
             </geometry>
         </collision>
-        <xacro:inertial_cylinder mass= "0.1" radius="0.0325" length="0.026">
-            <origin xyz="0.0 0.0 0.0" rpy="0.0 0.0 0.0"/>
+        <xacro:inertial_cylinder mass="${wheel_mass}" length="${wheel_thickness}" radius="${wheel_radius}">
+            <origin xyz="0 0 0" rpy="0 0 0"/>
         </xacro:inertial_cylinder>
     </link>
@@ -83,27 +96,25 @@
         <material>Gazebo/Blue</material>
     </gazebo>
-    <!-- right wheel -->
-    <joint name = "right_wheel_joint" type="continuous">
+    <!-- RIGHT WHEEL LINK -->
+    <joint name="right_wheel_joint" type="continuous">
         <parent link="base_link"/>
         <child link="right_wheel"/>
-        <origin xyz="0.0 -0.14 -0.07" rpy="${pi/2} 0.0 0.0"/>
-        <axis xyz="0.0 0.0 -1"/>
+        <origin xyz="0 ${-wheel_offset_y} 0" rpy="${pi/2} 0 0" />
+        <axis xyz="0 0 1"/>
     </joint>
     <link name="right_wheel">
         <visual>
-            <origin xyz="0 0 0"/>
             <geometry>
-                <cylinder radius="0.0325" length="0.026"/>
+                <cylinder radius="${wheel_radius}" length="${wheel_thickness}"/>
             </geometry>
             <material name="blue"/>
         </visual>
         <collision>
-            <origin xyz="0 0 0"/>
             <geometry>
-                <sphere radius="0.0325"/>
+                <sphere radius="${wheel_radius}"/>
             </geometry>
         </collision>
-        <xacro:inertial_cylinder mass= "0.1" radius="0.0325" length="0.026">
-            <origin xyz="0.0 0.0 0.0" rpy="0.0 0.0 0.0"/>
+        <xacro:inertial_cylinder mass="${wheel_mass}" length="${wheel_thickness}" radius="${wheel_radius}">
+            <origin xyz="0 0 0" rpy="0 0 0"/>
         </xacro:inertial_cylinder>
     </link>
@@ -111,59 +122,28 @@
         <material>Gazebo/Blue</material>
     </gazebo>
-<!-- front Castor wheel -->
-    <joint name="front_castor_wheel_joint" type="fixed">
+    <!-- CASTER WHEEL LINK -->
+    <joint name="caster_wheel_joint" type="fixed">
         <parent link="chassis"/>
-        <child link="front_castor_wheel"/>
-        <origin xyz="0.08 0.0 0.0" rpy="0.0 0.0 0.0"/>
+        <child link="caster_wheel"/>
+        <origin xyz="${caster_wheel_offset_x} 0 ${caster_wheel_offset_z}"/>
     </joint>
-    <link name="front_castor_wheel">
+    <link name="caster_wheel">
         <visual>
-            <origin xyz="0 0 0"/>
             <geometry>
-                <sphere radius="0.0325"/>
+                <sphere radius="${caster_wheel_radius}"/>
             </geometry>
-            <material name="black"/>
+            <material name="white"/>
         </visual>
         <collision>
-            <origin xyz="0 0 0"/>
             <geometry>
-                <sphere radius="0.0325"/>
+                <sphere radius="${caster_wheel_radius}"/>
             </geometry>
         </collision>
-        <xacro:inertial_sphere mass= "0.1" radius="0.0325">
-            <origin xyz="0.0 0.0 0.0" rpy="0.0 0.0 0.0"/>
+        <xacro:inertial_sphere mass="${caster_wheel_mass}" radius="${caster_wheel_radius}">
+            <origin xyz="0 0 0" rpy="0 0 0"/>
         </xacro:inertial_sphere>
     </link>
-    <gazebo reference="front_castor_wheel">
-        <material>Gazebo/Black</material>
-        <mu1 value="0.001"/>
-        <mu2 value="0.001"/>
-    </gazebo>
-    <!-- back Castor wheel -->
-    <joint name="back_castor_wheel_joint" type="fixed">
-        <parent link="chassis"/>
-        <child link="back_castor_wheel"/>
-        <origin xyz="-0.08 0.0 0.0" rpy="0.0 0.0 0.0"/>
-    </joint>
-    <link name="back_castor_wheel">
-        <visual>
-            <origin xyz="0 0 0"/>
-            <geometry>
-                <sphere radius="0.0325"/>
-            </geometry>
-            <material name="black"/>
-        </visual>
-        <collision>
-            <origin xyz="0 0 0"/>
-            <geometry>
-                <sphere radius="0.0325"/>
-            </geometry>
-        </collision>
-        <xacro:inertial_sphere mass= "0.1" radius="0.0325">
-            <origin xyz="0.0 0.0 0.0" rpy="0.0 0.0 0.0"/>
-        </xacro:inertial_sphere>
-    </link>
-    <gazebo reference="back_castor_wheel">
-        <material>Gazebo/Black</material>
+    <gazebo reference="caster_wheel">
+        <material>Gazebo/White</material>
         <mu1 value="0.001"/>
         <mu2 value="0.001"/>

File: dojo/description/ros2_control.xacro (robot description, xacro)
@@ -10,5 +10,6 @@
                 <param name="baud_rate">57600</param>
                 <param name="timeout">1000</param>
-                <param name="enc_counts_per_rev">1980</param>
+                <!-- <param name="enc_counts_per_rev">1980</param> -->
+                <param name="enc_counts_per_rev">1135</param>
             </hardware>
             <joint name="left_wheel_joint">
